File: BLE-DoorLock_v1_1/version_1_1.brd (EAGLE design)
At the start: 50 x 90 mm, 30 parts, among them Q1 MMBT2222, Q2 MMBT2222, Q3 DMN6140L

Commit message: First version for prototype PCB, 12VDC ONLY
Parts:
- added RESET1, RESET2, RESET3, RESET4, RESET5, RESET6: (no value), adafruit:1X01
- moved GPIO0 21.8 mm to (27.6, 59.9)
- moved 3V3 12.7 mm to (9.81, 80.2)
- moved R2 5.39 mm to (36.8, 52.1), turned to 180 degrees
- moved UART 2.54 mm to (44.5, 59.7)
- moved RESET 2.54 mm to (9.81, 75.1)
- moved Q2 1.27 mm to (33.0, 53.3)
- moved C1 1.27 mm to (30.5, 43.2)
- moved NCP1117 1.27 mm to (40.6, 45.7)
- moved R1 1.27 mm to (36.8, 55.9)
- turned R6 to 270 degrees
Connections:
- new net N$10: RESET4.1
- new net N$11: RESET5.1
- new net N$12: RESET6.1
- new net N$7: RESET1.1
- new net N$8: RESET2.1
- new net N$9: RESET3.1
- net RXD0: now also UART.5; no longer UART.4
- net TXD0: now also UART.4; no longer UART.5
Routing:
- net GND: track 6.84 -> 212.8 mm, vias 1 -> 2
- net GPIO0: track 47.2 -> 12.0 mm, vias 2 -> 0
- net +3V3: track 79.8 -> 108.3 mm, vias 4 -> 2
- net N$3: track 8.84 -> 1.89 mm
- net RTS: track 17.2 -> 11.0 mm, vias 2 -> 0
- net DTR: track 21.3 -> 25.4 mm, vias 0 -> 2
- net RXD0: track 25.2 -> 21.2 mm, vias 1 -> 0
- net RESET: track 83.0 -> 84.8 mm
- net GPIO13: track 18.5 -> 17.2 mm
- net N$2: track 2.98 -> 4.25 mm
- net +12V: track 52.8 -> 53.7 mm
- net N$6: track 3.98 -> 3.42 mm
- net TXD0: track 25.4 -> 25.6 mm, vias 1 -> 0
- removed copper zone on layer 1, net GND

Commit message: Before adding the relay
Parts:
- removed RESET1, RESET2, RESET3, RESET4, RESET5, RESET6: (no value), adafruit:1X01
Connections:
- removed net N$10: RESET4.1
- removed net N$11: RESET5.1
- removed net N$12: RESET6.1
- removed net N$7: RESET1.1
- removed net N$8: RESET2.1
- removed net N$9: RESET3.1
Changed lines of the file:
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@@
 <attribute name="MANUFACTURER_NAME" value="Phoenix Contact" x="34.29" y="7.62" size="1.778" layer="27" rot="R180" display="off"/>
 </element>
-<element name="RESET1" library="adafruit" package="1X01" value="" x="-22.86" y="-3.81"/>
-<element name="RESET2" library="adafruit" package="1X01" value="" x="-22.86" y="-8.89"/>
-<element name="RESET3" library="adafruit" package="1X01" value="" x="-22.86" y="-13.97"/>
-<element name="RESET4" library="adafruit" package="1X01" value="" x="-22.86" y="-19.05"/>
-<element name="RESET5" library="adafruit" package="1X01" value="" x="-22.86" y="-24.13"/>
-<element name="RESET6" library="adafruit" package="1X01" value="" x="-22.86" y="-29.21"/>
 </elements>
 <signals>
@@
 <wire x1="25.4" y1="50.8" x2="24.13" y2="52.07" width="0.4064" layer="1"/>
 </signal>
-<signal name="N$7">
-<contactref element="RESET1" pad="1"/>
-</signal>
-<signal name="N$8">
-<contactref element="RESET2" pad="1"/>
-</signal>
-<signal name="N$9">
-<contactref element="RESET3" pad="1"/>
-</signal>
-<signal name="N$10">
-<contactref element="RESET4" pad="1"/>
-</signal>
-<signal name="N$11">
-<contactref element="RESET5" pad="1"/>
-</signal>
-<signal name="N$12">
-<contactref element="RESET6" pad="1"/>
-</signal>
 </signals>
