File: BLE-DoorLock_v1_1/version_1_1.sch (EAGLE design)
At the start: 30 parts, among them Q1 MMBT2222, Q2 MMBT2222, Q3 DMN6140L

Commit message: First version for prototype PCB, 12VDC ONLY
Parts:
- added RESET1, RESET2, RESET3, RESET4, RESET5, RESET6: (no value), adafruit:PINHD-1X1
Connections:
- new net N$10: RESET4.1
- new net N$11: RESET5.1
- new net N$12: RESET6.1
- new net N$7: RESET1.1
- new net N$8: RESET2.1
- new net N$9: RESET3.1
- net RXD0: now also UART.5; no longer UART.4
- net TXD0: now also UART.4; no longer UART.5
Other:
- moved on the sheet: 12V, 3V3, GND, GPIO0, RESET

Commit message: Before adding the relay
Parts:
- removed RESET1, RESET2, RESET3, RESET4, RESET5, RESET6: (no value), adafruit:PINHD-1X1
Connections:
- removed net N$10: RESET4.1
- removed net N$11: RESET5.1
- removed net N$12: RESET6.1
- removed net N$7: RESET1.1
- removed net N$8: RESET2.1
- removed net N$9: RESET3.1
Changed lines of the file:
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@@
 <part name="DOOR-STRIKE" library="1729128" deviceset="1729128" device=""/>
 <part name="P+2" library="supply1" deviceset="+12V" device=""/>
-<part name="RESET1" library="adafruit" deviceset="PINHD-1X1" device=""/>
-<part name="RESET2" library="adafruit" deviceset="PINHD-1X1" device=""/>
-<part name="RESET3" library="adafruit" deviceset="PINHD-1X1" device=""/>
-<part name="RESET4" library="adafruit" deviceset="PINHD-1X1" device=""/>
-<part name="RESET5" library="adafruit" deviceset="PINHD-1X1" device=""/>
-<part name="RESET6" library="adafruit" deviceset="PINHD-1X1" device=""/>
 </parts>
 <sheets>
@@
 <instance part="DOOR-STRIKE" gate="G$1" x="180.34" y="35.56"/>
 <instance part="P+2" gate="1" x="177.8" y="43.18"/>
-<instance part="RESET1" gate="G$1" x="111.76" y="101.6" rot="MR0"/>
-<instance part="RESET2" gate="G$1" x="111.76" y="91.44" rot="MR0"/>
-<instance part="RESET3" gate="G$1" x="111.76" y="81.28" rot="MR0"/>
-<instance part="RESET4" gate="G$1" x="111.76" y="71.12" rot="MR0"/>
-<instance part="RESET5" gate="G$1" x="111.76" y="60.96" rot="MR0"/>
-<instance part="RESET6" gate="G$1" x="111.76" y="50.8" rot="MR0"/>
 </instances>
 <busses>
@@
 </segment>
 </net>
-<net name="N$7" class="0">
-<segment>
-<pinref part="RESET1" gate="G$1" pin="1"/>
-<wire x1="114.3" y1="101.6" x2="121.92" y2="101.6" width="0.1524" layer="91"/>
-</segment>
-</net>
-<net name="N$8" class="0">
-<segment>
-<pinref part="RESET2" gate="G$1" pin="1"/>
-<wire x1="114.3" y1="91.44" x2="121.92" y2="91.44" width="0.1524" layer="91"/>
-</segment>
-</net>
-<net name="N$9" class="0">
-<segment>
-<pinref part="RESET3" gate="G$1" pin="1"/>
-<wire x1="114.3" y1="81.28" x2="121.92" y2="81.28" width="0.1524" layer="91"/>
-</segment>
-</net>
-<net name="N$10" class="0">
-<segment>
-<pinref part="RESET4" gate="G$1" pin="1"/>
-<wire x1="114.3" y1="71.12" x2="121.92" y2="71.12" width="0.1524" layer="91"/>
-</segment>
-</net>
-<net name="N$11" class="0">
-<segment>
-<pinref part="RESET5" gate="G$1" pin="1"/>
-<wire x1="114.3" y1="60.96" x2="121.92" y2="60.96" width="0.1524" layer="91"/>
-</segment>
-</net>
-<net name="N$12" class="0">
-<segment>
-<pinref part="RESET6" gate="G$1" pin="1"/>
-<wire x1="114.3" y1="50.8" x2="121.92" y2="50.8" width="0.1524" layer="91"/>
-</segment>
-</net>
